File: 6col.kicad_pcb (KiCad board)
At the start: 2 copper layers, 135.3 x 94.8 mm, 51 parts, among them K1 KEYSW, K10 KEYSW, K11 KEYSW, K12 KEYSW, K13 KEYSW, K14 KEYSW, K15 KEYSW, K16 KEYSW, K17 KEYSW, K18 KEYSW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

Commit message: First version, looks ok
Parts:
- removed G*** (x2): LOGO, canadian_footprints:maple-8mm
- removed REF**: SolderWirePad_single_0-8mmDrill, Wire_Pads:SolderWirePad_single_0-8mmDrill
- K22: value TRRS -> TRRS_Through-Hole
Connections:
- D13 pad 2: Net-(D11-Pad2) (its old number) -> Net-(D13-Pad2)
- D14 pad 2: Net-(D11-Pad2) (its old number) -> Net-(D14-Pad2)
- D2 pad 2: Net-(D1-Pad2) -> Net-(D2-Pad2)
- D3 pad 2: Net-(D2-Pad2) -> Net-(D3-Pad2)
- D4 pad 2: Net-(D3-Pad2) -> Net-(D4-Pad2)
- D5 pad 2: Net-(D4-Pad2) -> Net-(D5-Pad2)
- D6 pad 2: Net-(D5-Pad2) -> Net-(D6-Pad2)
- D7 pad 2: Net-(D6-Pad2) -> Net-(D7-Pad2)
- D8 pad 2: Net-(D6-Pad2) -> Net-(D8-Pad2)
- K10 pad 1: /col3 -> /col4
- K11 pad 1: /col4 -> /col5
- K12 pad 1: /col5 -> /col6
- K13 pad 2: Net-(D11-Pad2) (its old number) -> Net-(D13-Pad2)
- K14 pad 1: /col1 -> /col2
- K14 pad 2: Net-(D11-Pad2) (its old number) -> Net-(D14-Pad2)
- K15 pad 1: /col2 -> /col3
- K16 pad 1: /col3 -> /col4
- K17 pad 1: /col4 -> /col5
- K18 pad 1: /col5 -> /col6
- K19 pad 1: /col3 -> /col4
- K20 pad 1: /col4 -> /col5
- K21 pad 1: /col5 -> /col6
- K6 pad 1: /col5 -> /col6
- K7 pad 2: Net-(D11-Pad2) (its old number) -> Net-(D7-Pad2)
- K8 pad 1: /col1 -> /col2
- K8 pad 2: Net-(D6-Pad2) -> Net-(D8-Pad2)
- K9 pad 1: /col2 -> /col3
- U1 pad 1: Net-(U1-Pad1) -> (no net)
- U1 pad 10: Net-(U1-Pad10) -> (no net)
- U1 pad 13: /col2 -> /col3
- U1 pad 14: /col3 -> /col4
- U1 pad 17: /col4 -> /col5
- U1 pad 19: /col5 -> /col6
- U1 pad 20: Net-(U1-Pad20) -> (no net)
- U1 pad 21: Net-(U1-Pad21) -> (no net)
- U1 pad 22: Net-(U1-Pad22) -> (no net)
- U1 pad 6: Net-(U1-Pad6) -> /col2
- U1 pad 7: Net-(U1-Pad7) -> (no net)
- U1 pad 8: Net-(U1-Pad8) -> (no net)
- U1 pad 9: Net-(U1-Pad9) -> (no net)
Routing:
- net /col6: track 0.00 -> 119.9 mm, vias 0 -> 2
- net /col3: track 76.4 -> 54.0 mm
- net /col5: track 119.9 -> 97.6 mm, vias 2 -> 1
- net /col4: track 97.4 -> 76.2 mm
- net /col1: track 56.7 -> 77.3 mm
- net /row3: track 93.5 -> 112.5 mm
- net /row2: track 84.4 -> 103.2 mm
- net /row1: track 82.6 -> 101.2 mm
- net Net-(D7-Pad2): track 0.00 -> 13.3 mm
- net Net-(D3-Pad2): track 6.35 -> 19.6 mm, vias 0 -> 1
- net Net-(D8-Pad2): track 0.00 -> 13.0 mm
- net Net-(D4-Pad2): track 13.0 -> 6.35 mm
- net Net-(D2-Pad2): track 19.6 -> 13.0 mm, vias 1 -> 0
- net Net-(D13-Pad2): track 0.00 -> 6.63 mm
- net Net-(D14-Pad2): track 0.00 -> 6.63 mm
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
Commit message: Fix TRRS soldermask and add missing pad
Parts:
- added REF**: SolderWirePad_single_0-8mmDrill, Wire_Pads:SolderWirePad_single_0-8mmDrill, F.Cu at (153.8, 68.1)
- K22: value TRRS_Through-Hole -> TRRS
Changed lines of the file:
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@@
     (tracks 323)
     (zones 0)
-    (modules 48)
+    (modules 49)
     (nets 39)
   )
@@
     (38 B.Mask user)
     (39 F.Mask user)
-    (40 Dwgs.User user)
-    (41 Cmts.User user)
-    (42 Eco1.User user)
-    (43 Eco2.User user)
+    (40 Dwgs.User user hide)
+    (41 Cmts.User user hide)
+    (42 Eco1.User user hide)
+    (43 Eco2.User user hide)
     (44 Edge.Cuts user)
     (45 Margin user)
-    (46 B.CrtYd user)
-    (47 F.CrtYd user)
-    (48 B.Fab user)
-    (49 F.Fab user)
+    (46 B.CrtYd user hide)
+    (47 F.CrtYd user hide)
+    (48 B.Fab user hide)
+    (49 F.Fab user hide)
   )
   (setup
@@
     (mod_text_size 1 1)
     (mod_text_width 0.15)
-    (pad_size 2.5 4.17)
-    (pad_drill 1.5)
+    (pad_size 1.99898 1.99898)
+    (pad_drill 1.0922)
     (pad_to_mask_clearance 0.2)
     (aux_axis_origin 0 0)
@@
     (add_net VCC)
   )
+  (module Wire_Pads:SolderWirePad_single_0-8mmDrill (layer F.Cu)
+    (at 153.77 68.14)
+    (fp_text reference REF** (at 0 -2.54) (layer F.SilkS) hide
+      (effects (font (size 1 1) (thickness 0.15)))
+    )
+    (fp_text value SolderWirePad_single_0-8mmDrill (at 0 2.54) (layer F.Fab)
+      (effects (font (size 1 1) (thickness 0.15)))
+    )
+    (pad 1 thru_hole circle (at 0 0) (size 1.99898 1.99898) (drill 1.0922) (layers *.Cu *.Mask)
+      (net 35 "Net-(K22-Pad2)"))
+  )
   (module canadian_footprints:Mx_Alps_100-dualside (layer F.Cu)
     (at 132.2625 125.73125)
@@
       (effects (font (size 1.524 1.778) (thickness 0.3048)))
     )
-    (fp_text value TRRS_Through-Hole (at 5.715 0) (layer F.SilkS)
+    (fp_text value TRRS (at 5.715 0) (layer F.SilkS)
       (effects (font (size 1.524 1.778) (thickness 0.3048)))
     )
@@
   (segment (start 166.62375 88.005) (end 166.62375 84.36125) (width 0.25) (layer F.Cu) (net 15) (status 20))
   (segment (start 167.11875 88.5) (end 166.62375 88.005) (width 0.25) (layer F.Cu) (net 15))
-  (segment (start 72.595 104.57) (end 71.375 105.79) (width 0.25) (layer B.Cu) (net 16))
-  (segment (start 77.5 104.57) (end 72.595 104.57) (width 0.25) (layer B.Cu) (net 16))
-  (segment (start 91.649062 104.567188) (end 90.42375 105.7925) (width 0.25) (layer B.Cu) (net 17))
-  (segment (start 96.54375 104.567188) (end 91.649062 104.567188) (width 0.25) (layer B.Cu) (net 17))
+  (segment (start 72.595 104.57) (end 71.375 105.79) (width 0.25) (layer B.Cu) (net 16) (status 20))
+  (segment (start 77.5 104.57) (end 72.595 104.57) (width 0.25) (layer B.Cu) (net 16) (status 10))
+  (segment (start 91.649062 104.567188) (end 90.42375 105.7925) (width 0.25) (layer B.Cu) (net 17) (status 20))
+  (segment (start 96.54375 104.567188) (end 91.649062 104.567188) (width 0.25) (layer B.Cu) (net 17) (status 10))
   (segment (start 110.564063 113.229688) (end 110.564063 105.945313) (width 0.25) (layer F.Cu) (net 18) (status 10))
   (segment (start 109.47375 104.855) (end 109.47375 101.03) (width 0.25) (layer F.Cu) (net 18) (status 20))
@@
   (segment (start 153 134.88125) (end 148.567902 134.88125) (width 0.25) (layer B.Cu) (net 20))
   (segment (start 154.996875 136.878125) (end 153 134.88125) (width 0.25) (layer B.Cu) (net 20))
-  (segment (start 142.020313 127.901563) (end 142.978125 127.901563) (width 0.25) (layer B.Cu) (net 20))
+  (segment (start 142.020313 127.901563) (end 142.978125 127.901563) (width 0.25) (layer B.Cu) (net 20) (status 20))
   (via (at 140.48 126.82) (size 0.6) (drill 0.4) (layers F.Cu B.Cu) (net 20))
   (segment (start 140.48 126.82) (end 142.020313 127.901563) (width 0.25) (layer B.Cu) (net 20))
   (segment (start 138.75 125.09) (end 140.48 126.82) (width 0.25) (layer F.Cu) (net 20))
   (segment (start 138.75 117.88125) (end 138.75 125.09) (width 0.25) (layer F.Cu) (net 20))
-  (segment (start 142.978125 133.251467) (end 145.164139 135.437481) (width 0.25) (layer F.Cu) (net 20))
-  (segment (start 142.978125 130.226563) (end 142.978125 133.251467) (width 0.25) (layer F.Cu) (net 20))
+  (segment (start 142.978125 133.251467) (end 145.164139 135.437481) (width 0.25) (layer F.Cu) (net 20) (status 20))
+  (segment (start 142.978125 130.226563) (end 142.978125 133.251467) (width 0.25) (layer F.Cu) (net 20) (status 10))
   (segment (start 148.06875 113.825) (end 148.06875 104.95) (width 0.25) (layer F.Cu) (net 21) (status 10))
   (segment (start 147.57375 104.455) (end 147.57375 101.03) (width 0.25) (layer F.Cu) (net 21) (status 20))
@@
   (segment (start 121.71375 79.59875) (end 121.71375 87.21375) (width 0.25) (layer F.Cu) (net 26) (status 10))
   (segment (start 121.71375 98.64875) (end 121.71375 106.96375) (width 0.25) (layer F.Cu) (net 26) (status 10))
-  (segment (start 128.71125 122.46125) (end 128.8575 122.46125) (width 0.25) (layer F.Cu) (net 26))
-  (segment (start 125.25 119) (end 128.71125 122.46125) (width 0.25) (layer F.Cu) (net 26))
+  (segment (start 128.71125 122.46125) (end 128.8575 122.46125) (width 0.25) (layer F.Cu) (net 26) (status 30))
+  (segment (start 125.25 119) (end 128.71125 122.46125) (width 0.25) (layer F.Cu) (net 26) (status 20))
   (segment (start 127.75 65.13125) (end 126.25 66.63125) (width 0.25) (layer B.Cu) (net 27))
   (segment (start 136.25 65.13125) (end 127.75 65.13125) (width 0.25) (layer B.Cu) (net 27))
@@
   (segment (start 114.358125 66.63125) (end 113.68875 65.961875) (width 0.25) (layer B.Cu) (net 27) (status 20))
   (segment (start 144.5 118.5) (end 144.5 120.2) (width 0.25) (layer F.Cu) (net 27))
-  (segment (start 148.372644 124.072644) (end 151.251111 124.072644) (width 0.25) (layer F.Cu) (net 27))
+  (segment (start 148.372644 124.072644) (end 151.251111 124.072644) (width 0.25) (layer F.Cu) (net 27) (status 20))
   (segment (start 144.5 120.2) (end 148.372644 124.072644) (width 0.25) (layer F.Cu) (net 27))
   (segment (start 113.68875 68.501875) (end 131.120625 68.501875) (width 0.25) (layer B.Cu) (net 28) (status 10))
@@
   (segment (start 133.35 59.23125) (end 131.25 57.13125) (width 0.25) (layer F.Cu) (net 31) (status 10))
   (segment (start 139.65 59.28125) (end 133.35 59.28125) (width 0.25) (layer F.Cu) (net 31) (status 30))
-  (segment (start 135.702187 122.426563) (end 135.6675 122.46125) (width 0.25) (layer F.Cu) (net 32))
-  (segment (start 135.702187 122.426563) (end 135.6675 122.46125) (width 0.25) (layer B.Cu) (net 32))
-  (segment (start 142.978125 122.426563) (end 135.702187 122.426563) (width 0.25) (layer B.Cu) (net 32))
+  (segment (start 135.702187 122.426563) (end 135.6675 122.46125) (width 0.25) (layer F.Cu) (net 32) (status 30))
+  (segment (start 135.702187 122.426563) (end 135.6675 122.46125) (width 0.25) (layer B.Cu) (net 32) (status 30))
+  (segment (start 142.978125 122.426563) (end 135.702187 122.426563) (width 0.25) (layer B.Cu) (net 32) (status 30))
   (segment (start 152.698361 137.456269) (end 152.698361 133.432889) (width 0.25) (layer F.Cu) (net 33) (status 10))
   (segment (start 157 129.13125) (end 157 126.664267) (width 0.25) (layer F.Cu) (net 33) (status 20))
@@
   (segment (start 176.121249 137.510001) (end 181.25 132.38125) (width 0.25) (layer F.Cu) (net 34))
   (segment (start 177.278684 125.909934) (end 176.376847 125.909934) (width 0.25) (layer F.Cu) (net 34) (status 30))
-  (segment (start 153.7716 68.1482) (end 153.7716 62.484) (width 0.25) (layer F.Cu) (net 35))
   (segment (start 153.7716 62.484) (end 153.797 62.4586) (width 0.25) (layer F.Cu) (net 35))
   (segment (start 152.186987 62.4586) (end 153.797 62.4586) (width 0.25) (layer F.Cu) (net 35))
@@
   (segment (start 150.08695 61.597838) (end 151.326225 61.597838) (width 0.25) (layer F.Cu) (net 35) (status 10))
   (segment (start 151.326225 61.597838) (end 152.186987 62.4586) (width 0.25) (layer F.Cu) (net 35))
+  (segment (start 153.7716 68.1482) (end 153.7716 62.484) (width 0.25) (layer F.Cu) (net 35))
   (segment (start 162.75 59.38125) (end 161.5 59.38125) (width 0.25) (layer B.Cu) (net 36) (status 10))
   (segment (start 159.962788 56.594038) (end 158.34195 56.594038) (width 0.25) (layer B.Cu) (net 36) (status 20))

Commit message: Add holes in pcb to use standoffs
Parts:
- added ?: , kbd:LEGO_HOLE, F.Cu at (153.1, 75.7)
- added ?: , kbd:LEGO_HOLE, F.Cu at (153.7, 112.8)
- added ?: , kbd:LEGO_HOLE, F.Cu at (115.0, 94.8)
- added ?: , kbd:LEGO_HOLE, F.Cu at (77.5, 99.5)
- added ?: , kbd:LEGO_HOLE, F.Cu at (77.5, 80.5)
Routing:
- net /row1: track 101.2 -> 112.0 mm
- net /row2: track 103.2 -> 110.2 mm
- net /row3: track 112.5 -> 117.3 mm
- net /row4: track 97.0 -> 98.6 mm

Commit message: Add creators
Other:
- board text added: "PCB Designed by: /u/That-Canadian LeReverandNox Grivel-l"
- board text removed: "PCB Designed by: /u/That-Canadian"
Changed lines of the file:
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@@
   (page A4)
   (layers
-    (0 F.Cu signal)
+    (0 F.Cu signal hide)
     (31 B.Cu signal)
     (32 B.Adhes user)
@@
       (net 25 /col3))
   )
+  (gr_text "PCB Designed by:\n/u/That-Canadian\nLeReverandNox\nGrivel-l" (at 180.85562 118.74246 330) (layer B.SilkS)
+    (effects (font (size 1 1) (thickness 0.15)) (justify mirror))
+  )
+  (gr_text "PCB Designed by:\n/u/That-Canadian\nLeReverandNox\nGrivel-l" (at 180.85562 118.74246 330) (layer F.SilkS)
+    (effects (font (size 1 1) (thickness 0.15)))
+  )
   (gr_text ProMicro (at 106.172 73.787) (layer B.SilkS)
     (effects (font (size 1.27 1.524) (thickness 0.2032)) (justify mirror))
@@
   )
   (gr_line (start 194.056 120.904) (end 194.056 50.038) (angle 90) (layer Dwgs.User) (width 0.2))
-  (gr_text "PCB Designed by:\n/u/That-Canadian" (at 181.25 118.63125 330) (layer B.SilkS)
-    (effects (font (size 1.5 1.5) (thickness 0.3)) (justify mirror))
-  )
-  (gr_text "PCB Designed by:\n/u/That-Canadian" (at 181.25 118.63125 330) (layer F.SilkS)
-    (effects (font (size 1.5 1.5) (thickness 0.3)))
-  )
   (gr_line (start 176.315625 148.948438) (end 160.8375 140.01875) (angle 90) (layer Edge.Cuts) (width 0.15))
   (gr_line (start 193.579688 122.159375) (end 178.101563 148.353125) (angle 90) (layer Edge.Cuts) (width 0.15))
